Commit message: simulation without correct foot control

File: simulation/pybullet/model/urdf/brutus.urdf (robot description, URDF)
Before this commit: robot brutus, 44 links, 43 joints
Links:
- link battery: mass 0.2 -> 0.0002

Commit message: need to relocate feet

File: simulation/pybullet/model/urdf/brutus.urdf (robot description, URDF)
Before this commit: robot brutus, 44 links, 43 joints
Links:
- link battery: mass 0.0002 -> 0.2
- link foot_link_bl: geometry collision mesh filename=../meshes/foot_fist_mesh.stl scale=0.001 0.001 0.001; visual mesh filename=../meshes/foot_fist_mesh.stl scale=0.001 0.001 0.001
- link foot_link_br: geometry collision mesh filename=../meshes/foot_fist_mesh.stl scale=0.001 0.001 0.001; visual mesh filename=../meshes/foot_fist_mesh.stl scale=0.001 0.001 0.001
- link foot_link_fl: geometry collision mesh filename=../meshes/foot_fist_mesh.stl scale=0.001 0.001 0.001; visual mesh filename=../meshes/foot_fist_mesh.stl scale=0.001 0.001 0.001
- link foot_link_fr: geometry collision mesh filename=../meshes/foot_fist_mesh.stl; visual mesh filename=../meshes/foot_fist_mesh.stl scale=0.001 0.001 0.001
- link up_box_link: mass 0.03146 -> 0.33146

Commit message: Changed to fist foot

File: simulation/pybullet/model/urdf/brutus.urdf (robot description, URDF)
Before this commit: robot brutus, 44 links, 43 joints
Links:
- link foot_link_bl: geometry collision mesh filename=../meshes/foot_fist_mesh_relocated.stl scale=0.001 0.001 0.001; visual mesh filename=../meshes/foot_fist_mesh_relocated.stl scale=0.001 0.001 0.001
- link foot_link_br: geometry collision mesh filename=../meshes/foot_fist_mesh_relocated.stl scale=0.001 0.001 0.001; visual mesh filename=../meshes/foot_fist_mesh_relocated.stl scale=0.001 0.001 0.001
- link foot_link_fl: geometry collision mesh filename=../meshes/foot_fist_mesh_relocated.stl scale=0.001 0.001 0.001; visual mesh filename=../meshes/foot_fist_mesh_relocated.stl scale=0.001 0.001 0.001
- link foot_link_fr: geometry collision mesh filename=../meshes/foot_fist_mesh_relocated.stl scale=0.001 0.001 0.001; visual mesh filename=../meshes/foot_fist_mesh_relocated.stl scale=0.001 0.001 0.001

Commit message: AAdded weight to chasis and box

File: simulation/pybullet/model/urdf/brutus.urdf (robot description, URDF)
Before this commit: robot brutus, 44 links, 43 joints
Links:
- link base_link: mass 0.00485 -> 0.0715
- link up_box_link: mass 0.33146 -> 0.65646

Commit message: Tried some changes (robot doesn't hold up)

File: simulation/pybullet/model/urdf/brutus.urdf (robot description, URDF)
Before this commit: robot brutus, 44 links, 43 joints
Joints:
- joint box_to_battery: origin xyz=-0.028 -0.035 0.005 rpy=0 0 0 -> xyz=0 0 0.0135 rpy=0 0 0

Commit message: Needs to check weights and movement angles

File: simulation/pybullet/model/urdf/brutus.urdf (robot description, URDF)
Before this commit: robot brutus, 44 links, 43 joints
Links:
- link up_box_link: mass 0.65646 -> 0.398

Commit message: changed mass values in urdf

File: simulation/pybullet/model/urdf/brutus.urdf (robot description, URDF)
Before this commit: robot brutus, 44 links, 43 joints
Links:
- link base_link: mass 0.0715 -> 0.04448
- link chasis_cover_link: mass 0.00335 -> 0.02205
- link foot_link_bl: mass 0.00294 -> 0.00946
- link foot_link_br: mass 0.00294 -> 0.00946
- link foot_link_fl: mass 0.00294 -> 0.00946
- link foot_link_fr: mass 0.00294 -> 0.00946
- link leg_bottom_link_bl: mass 0.00159 -> 0.00528
- link leg_bottom_link_br: mass 0.00159 -> 0.00528
- link leg_bottom_link_fl: mass 0.00159 -> 0.00528
- link leg_bottom_link_fr: mass 0.00159 -> 0.00528
- link leg_elbow_bl: mass 0.00282 -> 0.00985
- link leg_elbow_br: mass 0.00282 -> 0.00985
- link leg_elbow_fl: mass 0.00282 -> 0.00985
- link leg_elbow_fr: mass 0.00282 -> 0.00985
- link spacer_bl: mass 0.00004 -> 0.00036
- link spacer_br: mass 0.00004 -> 0.00036
- link spacer_fl: mass 0.00004 -> 0.00036
- link spacer_fr: mass 0.00004 -> 0.00036
- link up_box_link: mass 0.398 -> 0.38168
- link upper_link_bl: mass 0.000005 -> 0.00385
- link upper_link_br: mass 0.000005 -> 0.00385
- link upper_link_fl: mass 0.000005 -> 0.00385
- link upper_link_fr: mass 0.000005 -> 0.00385

Commit message: Added most of the project

File: simulation/pybullet/model/urdf/brutus.urdf (robot description, URDF)
Before this commit: robot brutus, 44 links, 43 joints
Links:
- link base_link: mass 0.00485 -> 0.04448
- link chasis_cover_link: mass 0.00335 -> 0.02205
- link foot_link_bl: mass 0.00294 -> 0.00946; geometry collision mesh filename=../meshes/foot_fist_mesh_relocated.stl scale=0.001 0.001 0.001; visual mesh filename=../meshes/foot_fist_mesh_relocated.stl scale=0.001 0.001 0.001
- link foot_link_br: mass 0.00294 -> 0.00946; geometry collision mesh filename=../meshes/foot_fist_mesh_relocated.stl scale=0.001 0.001 0.001; visual mesh filename=../meshes/foot_fist_mesh_relocated.stl scale=0.001 0.001 0.001
- link foot_link_fl: mass 0.00294 -> 0.00946; geometry collision mesh filename=../meshes/foot_fist_mesh_relocated.stl scale=0.001 0.001 0.001; visual mesh filename=../meshes/foot_fist_mesh_relocated.stl scale=0.001 0.001 0.001
- link foot_link_fr: mass 0.00294 -> 0.00946; geometry collision mesh filename=../meshes/foot_fist_mesh_relocated.stl scale=0.001 0.001 0.001; visual mesh filename=../meshes/foot_fist_mesh_relocated.stl scale=0.001 0.001 0.001
- link leg_bottom_link_bl: mass 0.00159 -> 0.00528
- link leg_bottom_link_br: mass 0.00159 -> 0.00528
- link leg_bottom_link_fl: mass 0.00159 -> 0.00528
- link leg_bottom_link_fr: mass 0.00159 -> 0.00528
- link leg_elbow_bl: mass 0.00282 -> 0.00985
- link leg_elbow_br: mass 0.00282 -> 0.00985
- link leg_elbow_fl: mass 0.00282 -> 0.00985
- link leg_elbow_fr: mass 0.00282 -> 0.00985
- link spacer_bl: mass 0.00004 -> 0.00036
- link spacer_br: mass 0.00004 -> 0.00036
- link spacer_fl: mass 0.00004 -> 0.00036
- link spacer_fr: mass 0.00004 -> 0.00036
- link up_box_link: mass 0.03146 -> 0.38168
- link upper_link_bl: mass 0.000005 -> 0.00385
- link upper_link_br: mass 0.000005 -> 0.00385
- link upper_link_fl: mass 0.000005 -> 0.00385
- link upper_link_fr: mass 0.000005 -> 0.00385
Joints:
- joint box_to_battery: origin xyz=-0.028 -0.035 0.005 rpy=0 0 0 -> xyz=0 0 0.0135 rpy=0 0 0
